File: hw/PCBDesign/DroneController.sch (KiCad schematic (older format))
At the start: 0 parts

Commit message: Clean up schematics some
Changed lines of the file:
@@
 $EndSheet
 $Sheet
-S 6850 4650 1150 1350
+S 6850 4650 1150 1650
 U 6045890B
 F0 "Wireless" 50
@@
 F12 "nRF24_IRQ" O L 6850 5900 50
 F13 "V+" I R 8000 4750 50
+F14 "BT_VCC_EN" I L 6850 6000 50
+F15 "RF24_VCC_EN" I L 6850 6100 50
 $EndSheet
 $Comp
@@
 $EndSheet
 $Sheet
-S 4500 1000 2000 5000
+S 4500 1000 2000 5300
 U 604707FB
 F0 "Processor" 50
@@
 F25 "EEPROM_SDA" B R 6500 4050 50
 F26 "EEPROM_SCL" O R 6500 4150 50
-F27 "VSense_USB" I L 4500 2500 50
 F28 "VSense_Digital" I L 4500 2600 50
 F29 "VSense_Radio" I L 4500 2700 50
@@
 F31 "V+" I L 4500 2250 50
 F32 "nRESET" I R 6500 3000 50
-F33 "nBOOT" I R 6500 2900 50
 F34 "PWM_Buzzer" O R 6500 1100 50
 F35 "KEY_MOSI" O R 6500 1300 50
@@
 F46 "ANALOG_IN_VYAW" I R 6500 2600 50
 F47 "ANALOG_IN_VTHROTTLE" I R 6500 2700 50
+F48 "VDDA" I L 4500 2150 50
+F49 "DBG_UART_TX" O L 4500 3600 50
+F50 "DBG_UART_RX" I L 4500 3700 50
+F51 "BT_VCC_EN" O R 6500 6000 50
+F52 "RF24_VCC_EN" O R 6500 6100 50
 $EndSheet
 $Comp
@@
 	6500 4150 6850 4150
 $Comp
-L power:+5V #PWR?
-U 1 1 6064DADB
-P 4350 2500
-F 0 "#PWR?" H 4350 2350 50  0001 C CNN
-F 1 "+5V" V 4350 2700 50  0000 C CNN
-F 2 "" H 4350 2500 50  0001 C CNN
-F 3 "" H 4350 2500 50  0001 C CNN
-	1    4350 2500
-	0    -1   -1   0
-$EndComp
-$Comp
 L power:+3V3 #PWR?
 U 1 1 6064DFA8
@@
 $EndComp
 Wire Wire Line
-	4350 2500 4500 2500
-Wire Wire Line
 	4350 2600 4500 2600
 Wire Wire Line
@@
 Wire Wire Line
 	6500 2200 6850 2200
+$Comp
+L power:+3.3VADC #PWR?
+U 1 1 60499637
+P 4350 2150
+F 0 "#PWR?" H 4500 2100 50  0001 C CNN
+F 1 "+3.3VADC" V 4350 2450 50  0000 C CNN
+F 2 "" H 4350 2150 50  0001 C CNN
+F 3 "" H 4350 2150 50  0001 C CNN
+	1    4350 2150
+	0    -1   -1   0
+$EndComp
+Wire Wire Line
+	4350 2150 4500 2150
+Wire Wire Line
+	6500 6000 6850 6000
+Wire Wire Line
+	6500 6100 6850 6100
 $EndSCHEMATC

Commit message: Schematic polishing
Parts:
- added J1: SerialDebug, Connector_PinHeader_2.54mm:PinHeader_1x02_P2.54mm_Vertical, symbol Connector_Generic:Conn_01x02
Connections:
- net Processor/DBG_UART_RX: now also J1.2 (Pin_2)
- net Processor/DBG_UART_TX: now also J1.1 (Pin_1)
Changed lines of the file:
@@
 F1 "HMIHardware.sch" 50
 F2 "PWM_Buzzer" I L 6850 1100 50
-F3 "KEY_MOSI" I L 6850 1300 50
 F4 "KEY_MISO" O L 6850 1400 50
 F5 "KEY_SCK" O L 6850 1500 50
@@
 F15 "JS_VT" O L 6850 2700 50
 F16 "V+" O R 8000 1100 50
-F17 "nBOOT" O L 6850 2900 50
 F18 "nRESET" O L 6850 3000 50
 $EndSheet
@@
 $EndSheet
 $Comp
-L power:+5V #PWR?
+L power:+5V #PWR01
 U 1 1 605EF5C1
 P 2750 4900
-F 0 "#PWR?" H 2750 4750 50  0001 C CNN
+F 0 "#PWR01" H 2750 4750 50  0001 C CNN
 F 1 "+5V" V 2750 5100 50  0000 C CNN
 F 2 "" H 2750 4900 50  0001 C CNN
@@
 $EndComp
 $Comp
-L power:+3V3 #PWR?
+L power:+3V3 #PWR02
 U 1 1 6061DB0D
 P 2750 5050
-F 0 "#PWR?" H 2750 4900 50  0001 C CNN
+F 0 "#PWR02" H 2750 4900 50  0001 C CNN
 F 1 "+3V3" V 2750 5250 50  0000 C CNN
 F 2 "" H 2750 5050 50  0001 C CNN
@@
 $EndComp
 $Comp
-L power:+3.3VADC #PWR?
+L power:+3.3VADC #PWR03
 U 1 1 6061E3DE
 P 2750 5200
-F 0 "#PWR?" H 2900 5150 50  0001 C CNN
+F 0 "#PWR03" H 2900 5150 50  0001 C CNN
 F 1 "+3.3VADC" V 2750 5500 50  0000 C CNN
 F 2 "" H 2750 5200 50  0001 C CNN
@@
 $EndComp
 $Comp
-L power:+3.3VP #PWR?
+L power:+3.3VP #PWR04
 U 1 1 6061E741
 P 2750 5350
-F 0 "#PWR?" H 2900 5300 50  0001 C CNN
+F 0 "#PWR04" H 2900 5300 50  0001 C CNN
 F 1 "+3.3VP" V 2750 5600 50  0000 C CNN
 F 2 "" H 2750 5350 50  0001 C CNN
@@
 F25 "EEPROM_SDA" B R 6500 4050 50
 F26 "EEPROM_SCL" O R 6500 4150 50
-F28 "VSense_Digital" I L 4500 2600 50
-F29 "VSense_Radio" I L 4500 2700 50
-F30 "VSense_Analog" I L 4500 2800 50
-F31 "V+" I L 4500 2250 50
-F32 "nRESET" I R 6500 3000 50
-F34 "PWM_Buzzer" O R 6500 1100 50
-F35 "KEY_MOSI" O R 6500 1300 50
-F36 "KEY_MISO" I R 6500 1400 50
-F37 "KEY_SCK" O R 6500 1500 50
-F38 "KEY_nCS" O R 6500 1600 50
-F39 "KEY_nSAMPLE" O R 6500 1700 50
-F40 "ENCODER0_A" I R 6500 1900 50
-F41 "ENCODER0_B" I R 6500 2000 50
-F42 "ENCODER1_A" I R 6500 2100 50
-F43 "ENCODER1_B" I R 6500 2200 50
-F44 "ANALOG_IN_VPITCH" I R 6500 2400 50
-F45 "ANALOG_IN_VROLL" I R 6500 2500 50
-F46 "ANALOG_IN_VYAW" I R 6500 2600 50
-F47 "ANALOG_IN_VTHROTTLE" I R 6500 2700 50
-F48 "VDDA" I L 4500 2150 50
-F49 "DBG_UART_TX" O L 4500 3600 50
-F50 "DBG_UART_RX" I L 4500 3700 50
-F51 "BT_VCC_EN" O R 6500 6000 50
-F52 "RF24_VCC_EN" O R 6500 6100 50
-$EndSheet
-$Comp
-L power:+3.3VP #PWR?
+F27 "VSense_Digital" I L 4500 2600 50
+F28 "VSense_Radio" I L 4500 2700 50
+F29 "VSense_Analog" I L 4500 2800 50
+F30 "V+" I L 4500 2250 50
+F31 "nRESET" I R 6500 3000 50
+F32 "PWM_Buzzer" O R 6500 1100 50
+F33 "KEY_MOSI" O R 6500 1300 50
+F34 "KEY_MISO" I R 6500 1400 50
+F35 "KEY_SCK" O R 6500 1500 50
+F36 "KEY_nCS" O R 6500 1600 50
+F37 "KEY_nSAMPLE" O R 6500 1700 50
+F38 "ENCODER0_A" I R 6500 1900 50
+F39 "ENCODER0_B" I R 6500 2000 50
+F40 "ENCODER1_A" I R 6500 2100 50
+F41 "ENCODER1_B" I R 6500 2200 50
+F42 "ANALOG_IN_VPITCH" I R 6500 2400 50
+F43 "ANALOG_IN_VROLL" I R 6500 2500 50
+F44 "ANALOG_IN_VYAW" I R 6500 2600 50
+F45 "ANALOG_IN_VTHROTTLE" I R 6500 2700 50
+F46 "VDDA" I L 4500 2150 50
+F47 "DBG_UART_TX" O L 4500 3600 50
+F48 "DBG_UART_RX" I L 4500 3700 50
+F49 "BT_VCC_EN" O R 6500 6000 50
+F50 "RF24_VCC_EN" O R 6500 6100 50
+$EndSheet
+$Comp
+L power:+3.3VP #PWR012
 U 1 1 606332FD
 P 8150 4750
-F 0 "#PWR?" H 8300 4700 50  0001 C CNN
+F 0 "#PWR012" H 8300 4700 50  0001 C CNN
 F 1 "+3.3VP" V 8150 5000 50  0000 C CNN
 F 2 "" H 8150 4750 50  0001 C CNN
@@
 	4050 5850 4500 5850
 $Comp
-L power:+3V3 #PWR?
+L power:+3V3 #PWR011
 U 1 1 60647C04
 P 8150 3550
-F 0 "#PWR?" H 8150 3400 50  0001 C CNN
+F 0 "#PWR011" H 8150 3400 50  0001 C CNN
 F 1 "+3V3" V 8150 3750 50  0000 C CNN
 F 2 "" H 8150 3550 50  0001 C CNN
@@
 	6500 4150 6850 4150
 $Comp
-L power:+3V3 #PWR?
+L power:+3V3 #PWR07
 U 1 1 6064DFA8
 P 4350 2600
-F 0 "#PWR?" H 4350 2450 50  0001 C CNN
+F 0 "#PWR07" H 4350 2450 50  0001 C CNN
 F 1 "+3V3" V 4350 2800 50  0000 C CNN
 F 2 "" H 4350 2600 50  0001 C CNN
@@
 $EndComp
 $Comp
-L power:+3.3VADC #PWR?
+L power:+3.3VADC #PWR09
 U 1 1 6064E61E
 P 4350 2800
-F 0 "#PWR?" H 4500 2750 50  0001 C CNN
+F 0 "#PWR09" H 4500 2750 50  0001 C CNN
 F 1 "+3.3VADC" V 4350 3100 50  0000 C CNN
 F 2 "" H 4350 2800 50  0001 C CNN
@@
 $EndComp
 $Comp
-L power:+3.3VP #PWR?
+L power:+3.3VP #PWR08
 U 1 1 6064E986
 P 4350 2700
-F 0 "#PWR?" H 4500 2650 50  0001 C CNN
+F 0 "#PWR08" H 4500 2650 50  0001 C CNN
 F 1 "+3.3VP" V 4350 2950 50  0000 C CNN
 F 2 "" H 4350 2700 50  0001 C CNN
@@
 	4350 2800 4500 2800
 $Comp
-L power:+3V3 #PWR?
+L power:+3V3 #PWR06
 U 1 1 60655154
 P 4350 2250
-F 0 "#PWR?" H 4350 2100 50  0001 C CNN
+F 0 "#PWR06" H 4350 2100 50  0001 C CNN
 F 1 "+3V3" V 4350 2450 50  0000 C CNN
 F 2 "" H 4350 2250 50  0001 C CNN
@@
 	4350 2250 4500 2250
 $Comp
-L power:+3V3 #PWR?
+L power:+3V3 #PWR010
 U 1 1 60656218
 P 8150 1100
-F 0 "#PWR?" H 8150 950 50  0001 C CNN
+F 0 "#PWR010" H 8150 950 50  0001 C CNN
 F 1 "+3V3" V 8150 1300 50  0000 C CNN
 F 2 "" H 8150 1100 50  0001 C CNN
@@
 	8150 1100 8000 1100
 Wire Wire Line
-	6500 2900 6850 2900
-Wire Wire Line
 	6500 3000 6850 3000
 Wire Wire Line
@@
 	6500 1100 6850 1100
 Wire Wire Line
-	6500 1300 6850 1300
-Wire Wire Line
 	6500 1400 6850 1400
 Wire Wire Line
@@
 	6500 2200 6850 2200
 $Comp
-L power:+3.3VADC #PWR?
+L power:+3.3VADC #PWR05
 U 1 1 60499637
 P 4350 2150
-F 0 "#PWR?" H 4500 2100 50  0001 C CNN
+F 0 "#PWR05" H 4500 2100 50  0001 C CNN
 F 1 "+3.3VADC" V 4350 2450 50  0000 C CNN
 F 2 "" H 4350 2150 50  0001 C CNN
@@
 Wire Wire Line
 	6500 6100 6850 6100
+$Comp
+L Connector_Generic:Conn_01x02 J1
+U 1 1 604BEF1D
+P 4100 3600
+F 0 "J1" H 4018 3817 50  0000 C CNN
+F 1 "SerialDebug" H 4018 3726 50  0000 C CNN
+F 2 "Connector_PinHeader_2.54mm:PinHeader_1x02_P2.54mm_Vertical" H 4100 3600 50  0001 C CNN
+F 3 "~" H 4100 3600 50  0001 C CNN
+	1    4100 3600
+	-1   0    0    -1
+$EndComp
+Wire Wire Line
+	4300 3600 4500 3600
+Wire Wire Line
+	4300 3700 4500 3700
 $EndSCHEMATC

Commit message: Update pcb
Parts:
- added H1, H2, H3, H4: MountingHole_Pad, MountingHole:MountingHole_3.2mm_M3_Pad_Via, symbol Mechanical:MountingHole_Pad
Connections:
- new net GND: H1.1, H2.1, H3.1, H4.1
Changed lines of the file:
@@
 Wire Wire Line
 	4300 3700 4500 3700
+$Comp
+L Mechanical:MountingHole_Pad H1
+U 1 1 60507987
+P 1000 1050
+F 0 "H1" H 1100 1099 50  0000 L CNN
+F 1 "MountingHole_Pad" H 1100 1008 50  0000 L CNN
+F 2 "MountingHole:MountingHole_3.2mm_M3_Pad_Via" H 1000 1050 50  0001 C CNN
+F 3 "~" H 1000 1050 50  0001 C CNN
+	1    1000 1050
+	1    0    0    -1
+$EndComp
+$Comp
+L power:GND #PWR0114
+U 1 1 60507F24
+P 1000 1150
+F 0 "#PWR0114" H 1000 900 50  0001 C CNN
+F 1 "GND" H 1005 977 50  0000 C CNN
+F 2 "" H 1000 1150 50  0001 C CNN
+F 3 "" H 1000 1150 50  0001 C CNN
+	1    1000 1150
+	1    0    0    -1
+$EndComp
+$Comp
+L Mechanical:MountingHole_Pad H2
+U 1 1 6050ADDB
+P 1000 1550
+F 0 "H2" H 1100 1599 50  0000 L CNN
+F 1 "MountingHole_Pad" H 1100 1508 50  0000 L CNN
+F 2 "MountingHole:MountingHole_3.2mm_M3_Pad_Via" H 1000 1550 50  0001 C CNN
+F 3 "~" H 1000 1550 50  0001 C CNN
+	1    1000 1550
+	1    0    0    -1
+$EndComp
+$Comp
+L power:GND #PWR0115
+U 1 1 6050ADE1
+P 1000 1650
+F 0 "#PWR0115" H 1000 1400 50  0001 C CNN
+F 1 "GND" H 1005 1477 50  0000 C CNN
+F 2 "" H 1000 1650 50  0001 C CNN
+F 3 "" H 1000 1650 50  0001 C CNN
+	1    1000 1650
+	1    0    0    -1
+$EndComp
+$Comp
+L Mechanical:MountingHole_Pad H3
+U 1 1 6050CE46
+P 1000 2050
+F 0 "H3" H 1100 2099 50  0000 L CNN
+F 1 "MountingHole_Pad" H 1100 2008 50  0000 L CNN
+F 2 "MountingHole:MountingHole_3.2mm_M3_Pad_Via" H 1000 2050 50  0001 C CNN
+F 3 "~" H 1000 2050 50  0001 C CNN
+	1    1000 2050
+	1    0    0    -1
+$EndComp
+$Comp
+L power:GND #PWR0116
+U 1 1 6050CE4C
+P 1000 2150
+F 0 "#PWR0116" H 1000 1900 50  0001 C CNN
+F 1 "GND" H 1005 1977 50  0000 C CNN
+F 2 "" H 1000 2150 50  0001 C CNN
+F 3 "" H 1000 2150 50  0001 C CNN
+	1    1000 2150
+	1    0    0    -1
+$EndComp
+$Comp
+L Mechanical:MountingHole_Pad H4
+U 1 1 6050EC15
+P 1000 2550
+F 0 "H4" H 1100 2599 50  0000 L CNN
+F 1 "MountingHole_Pad" H 1100 2508 50  0000 L CNN
+F 2 "MountingHole:MountingHole_3.2mm_M3_Pad_Via" H 1000 2550 50  0001 C CNN
+F 3 "~" H 1000 2550 50  0001 C CNN
+	1    1000 2550
+	1    0    0    -1
+$EndComp
+$Comp
+L power:GND #PWR0117
+U 1 1 6050EC1B
+P 1000 2650
+F 0 "#PWR0117" H 1000 2400 50  0001 C CNN
+F 1 "GND" H 1005 2477 50  0000 C CNN
+F 2 "" H 1000 2650 50  0001 C CNN
+F 3 "" H 1000 2650 50  0001 C CNN
+	1    1000 2650
+	1    0    0    -1
+$EndComp
 $EndSCHEMATC

Commit message: Lay out more PCB
Changed lines of the file:
@@
 F0 "Wireless" 50
 F1 "Wireless.sch" 50
-F2 "BT_INT_REQ" O L 6850 5000 50
-F3 "nBT_WAKEUP" I L 6850 5100 50
-F4 "nBT_PWR_UP" I L 6850 5200 50
 F5 "BT_RX" I L 6850 4850 50
 F6 "BT_TX" O L 6850 4750 50
@@
 	0    -1   -1   0
 $EndComp
-$Comp
-L power:+3.3VADC #PWR03
-U 1 1 6061E3DE
-P 2750 5200
-F 0 "#PWR03" H 2900 5150 50  0001 C CNN
-F 1 "+3.3VADC" V 2750 5500 50  0000 C CNN
-F 2 "" H 2750 5200 50  0001 C CNN
-F 3 "" H 2750 5200 50  0001 C CNN
-	1    2750 5200
-	0    -1   -1   0
-$EndComp
-$Comp
-L power:+3.3VP #PWR04
-U 1 1 6061E741
-P 2750 5350
-F 0 "#PWR04" H 2900 5300 50  0001 C CNN
-F 1 "+3.3VP" V 2750 5600 50  0000 C CNN
-F 2 "" H 2750 5350 50  0001 C CNN
-F 3 "" H 2750 5350 50  0001 C CNN
-	1    2750 5350
-	0    -1   -1   0
-$EndComp
 Wire Wire Line
 	2750 4900 2850 4900
 Wire Wire Line
 	2750 5050 2850 5050
-Wire Wire Line
-	2750 5200 2850 5200
-Wire Wire Line
-	2750 5350 2850 5350
 $Sheet
 S 2850 4800 1200 1200
@@
 F1 "PowerSupply.sch" 50
 F2 "V_Digital" B L 2850 5050 50
-F3 "V_Analog" B L 2850 5200 50
-F4 "V_Wireless" B L 2850 5350 50
 F5 "USB_D+" B R 4050 4950 50
 F6 "USB_D-" B R 4050 5050 50
@@
 F4 "nBatt_Pwr_Good" I L 4500 5250 50
 F5 "nBatt_Chg_Good" I L 4500 5350 50
-F6 "vBatt_Sense" I L 4500 5450 50
 F7 "nBattChgEn" O L 4500 5650 50
 F8 "BattChgCfg0" O L 4500 5750 50
@@
 F10 "BT_UART_RX" I R 6500 4750 50
 F11 "BT_UART_TX" O R 6500 4850 50
-F12 "BT_nWakeup" O R 6500 5100 50
-F13 "BT_nPowerUp" O R 6500 5200 50
-F14 "BT_IRQ" I R 6500 5000 50
 F15 "RF24_MOSI" O R 6500 5400 50
 F16 "RF24_MISO" I R 6500 5500 50
@@
 F26 "EEPROM_SCL" O R 6500 4150 50
 F27 "VSense_Digital" I L 4500 2600 50
-F28 "VSense_Radio" I L 4500 2700 50
-F29 "VSense_Analog" I L 4500 2800 50
 F30 "V+" I L 4500 2250 50
 F31 "nRESET" I R 6500 3000 50
@@
 F50 "RF24_VCC_EN" O R 6500 6100 50
 $EndSheet
-$Comp
-L power:+3.3VP #PWR012
-U 1 1 606332FD
-P 8150 4750
-F 0 "#PWR012" H 8300 4700 50  0001 C CNN
-F 1 "+3.3VP" V 8150 5000 50  0000 C CNN
-F 2 "" H 8150 4750 50  0001 C CNN
-F 3 "" H 8150 4750 50  0001 C CNN
-	1    8150 4750
-	0    1    1    0
-$EndComp
 Wire Wire Line
 	8150 4750 8000 4750
@@
 Wire Wire Line
 	6500 4850 6850 4850
-Wire Wire Line
-	6500 5000 6850 5000
-Wire Wire Line
-	6500 5100 6850 5100
-Wire Wire Line
-	6500 5200 6850 5200
 Wire Wire Line
 	6500 5400 6850 5400
@@
 	0    -1   -1   0
 $EndComp
-$Comp
-L power:+3.3VADC #PWR09
-U 1 1 6064E61E
-P 4350 2800
-F 0 "#PWR09" H 4500 2750 50  0001 C CNN
-F 1 "+3.3VADC" V 4350 3100 50  0000 C CNN
-F 2 "" H 4350 2800 50  0001 C CNN
-F 3 "" H 4350 2800 50  0001 C CNN
-	1    4350 2800
-	0    -1   -1   0
-$EndComp
-$Comp
-L power:+3.3VP #PWR08
-U 1 1 6064E986
-P 4350 2700
-F 0 "#PWR08" H 4500 2650 50  0001 C CNN
-F 1 "+3.3VP" V 4350 2950 50  0000 C CNN
-F 2 "" H 4350 2700 50  0001 C CNN
-F 3 "" H 4350 2700 50  0001 C CNN
-	1    4350 2700
-	0    -1   -1   0
-$EndComp
 Wire Wire Line
 	4350 2600 4500 2600
-Wire Wire Line
-	4350 2700 4500 2700
-Wire Wire Line
-	4350 2800 4500 2800
 $Comp
 L power:+3V3 #PWR06
@@
 $EndComp
 Wire Wire Line
-	4350 2250 4500 2250
+	4350 2250 4400 2250
 $Comp
 L power:+3V3 #PWR010
@@
 Wire Wire Line
 	6500 2200 6850 2200
-$Comp
-L power:+3.3VADC #PWR05
-U 1 1 60499637
-P 4350 2150
-F 0 "#PWR05" H 4500 2100 50  0001 C CNN
-F 1 "+3.3VADC" V 4350 2450 50  0000 C CNN
-F 2 "" H 4350 2150 50  0001 C CNN
-F 3 "" H 4350 2150 50  0001 C CNN
-	1    4350 2150
-	0    -1   -1   0
-$EndComp
-Wire Wire Line
-	4350 2150 4500 2150
 Wire Wire Line
 	6500 6000 6850 6000
@@
 	1    0    0    -1
 $EndComp
+$Comp
+L power:+3V3 #PWR0132
+U 1 1 6070E31F
+P 8150 4750
+F 0 "#PWR0132" H 8150 4600 50  0001 C CNN
+F 1 "+3V3" V 8150 4950 50  0000 C CNN
+F 2 "" H 8150 4750 50  0001 C CNN
+F 3 "" H 8150 4750 50  0001 C CNN
+	1    8150 4750
+	0    1    1    0
+$EndComp
+Wire Wire Line
+	4500 2150 4400 2150
+Wire Wire Line
+	4400 2150 4400 2250
+Connection ~ 4400 2250
+Wire Wire Line
+	4400 2250 4500 2250
 $EndSCHEMATC
