File: hw/PCBDesign/ButtonInput.sch (KiCad schematic (older format))
At the start: 31 parts

Commit message: Schematic polishing
Parts:
- C26, C27, C28, C29, C30, C31, C32, C33: renamed from C?; footprint (none) -> Capacitor_SMD:C_0402_1005Metric; LCSC (none) -> C1525
- R45, R47, R48, R51, R54, R55, R58: renamed from R?; footprint (none) -> Resistor_SMD:R_0402_1005Metric; LCSC (none) -> C11702
- R46, R49, R50, R52, R53, R56, R57, R59: renamed from R?; footprint (none) -> Resistor_SMD:R_0402_1005Metric; LCSC (none) -> C25744
- gave numbers to parts that had none: 8

Commit message: Added PCB
Parts:
- removed C26, C27, C29, C31, C33: 100n, Capacitor_SMD:C_0402_1005Metric, symbol Device:C
- removed R45, R47, R51, R54, R58: 1k, Resistor_SMD:R_0402_1005Metric, symbol Device:R_US
- removed R46, R49, R52, R56, R59: 10k, Resistor_SMD:R_0402_1005Metric, symbol Device:R_US
- removed SW11: Key_Left, symbol Switch:SW_Push
- removed SW12: Key_Right, symbol Switch:SW_Push
- removed SW14: Key_Up, symbol Switch:SW_Push
- removed SW16: Key_Down, symbol Switch:SW_Push
- removed SW18: Key_Enter, symbol Switch:SW_Push
- SW13: value Key_Esc -> Key_User; footprint (none) -> Button_Switch_SMD:SW_SPST_PTS810; DigiKey (none) -> CKN10504CT-ND
- SW15, SW17: footprint (none) -> Button_Switch_SMD:SW_SPST_PTS810; DigiKey (none) -> CKN10504CT-ND
Connections:
- net KeyEscape renamed KeyUser
Other:
- moved on the sheet: C28, C30, C32, R48, R50, R53, R55, R57, SW13, SW15, SW17
