File: hw/PCBDesign/DroneController.kicad_pcb (KiCad board)
At the start: 4 copper layers, 50 x 50 mm, 177 parts, among them J1 SerialDebug, J10 SW_B, J11 YTrim, J12 SW_C, J13 TTrim, J14 SW_D, J15 Conn_01x08, J2 USB_B_Micro, J3 SerialDebug, J4 Conn_ARM_JTAG_SWD_10, J5 EncoderConn, J6 JoystickConn, J7 PTrim, J8 SW_A, J9 RTrim, Q1 MMBT3904, Q2 MMBT3904, Q3 2N7002, Q5 LBSS84LT1G, SW13 Key_User, SW15 Key_nRESET, SW17 Key_nBOOT, U1 74HC165, U11 74HC595, U13 STM32F446RETx, U2 74HC165, U3 74HC165, U4 AT25SF081, U5 AT24C256, U8 AMS1117-3.3

Commit message: Add more of the I2C driver
Parts:
- J4: moved to B.Cu
- moved C57 54.9 mm to (124.2, 108.0)
- moved J4 52.0 mm to (104.4, 108.5), turned to 180 degrees
- moved C2 50.4 mm to (141.9, 100.0), turned to 180 degrees
- moved R96 44.2 mm to (124.0, 114.7), turned to 180 degrees
- moved R92 40.4 mm to (122.9, 101.5), turned to 270 degrees
- moved C55 39.5 mm to (133.1, 101.3), turned to 225 degrees
- moved C31 39.5 mm to (130.9, 116.8), turned to 45 degrees
- moved R65 39.3 mm to (140.2, 116.8), turned to 0 degrees
- moved D3 39.2 mm to (120.8, 101.4), turned to 0 degrees
- moved C56 39.1 mm to (138.7, 112.4), turned to 225 degrees
- moved C52 38.3 mm to (135.7, 100.8), turned to 225 degrees
- moved R97 36.8 mm to (136.0, 115.1), turned to 225 degrees
- moved C29 35.9 mm to (133.1, 116.8), turned to 135 degrees
- moved R67 33.8 mm to (134.2, 97.0), turned to 0 degrees
- moved R89 33.2 mm to (140.2, 114.8), turned to 0 degrees
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Connections:
- U13 pad 10: /Processor/ANALOG_IN_VTHROTTLE -> /Processor/ANALOG_IN_VPITCH
- U13 pad 11: /Processor/ANALOG_IN_VYAW -> /Processor/ANALOG_IN_VROLL
- U13 pad 8: /Processor/ANALOG_IN_VROLL -> /Processor/ANALOG_IN_VTHROTTLE
- U13 pad 9: /Processor/ANALOG_IN_VPITCH -> /Processor/ANALOG_IN_VYAW
Routing:
- net /Human Machine Interface/KEY_nCS: track 1.65 -> 38.3 mm, vias 0 -> 3
- net /Processor/RF24_nIRQ: track 1.48 -> 36.7 mm, vias 0 -> 2
- net /Processor/RF24_nCS: track 1.48 -> 34.4 mm, vias 0 -> 2
- net /Processor/RF24_CE: track 0.00 -> 31.2 mm, vias 0 -> 2
- net /Processor/RF24_SCK: track 0.00 -> 29.9 mm, vias 0 -> 2
- net /Processor/RF24_MISO: track 0.00 -> 28.8 mm, vias 0 -> 2
- net /Processor/RF24_MOSI: track 0.00 -> 28.6 mm, vias 0 -> 2
- net /Power Supply/USB_ID: track 3.42 -> 22.9 mm, vias 0 -> 2
- net /Power Supply/USB_D+: track 4.56 -> 22.4 mm, vias 0 -> 2
- net /Processor/USB_SENSE: track 0.00 -> 17.1 mm, vias 0 -> 2
- net /Power Supply/USB_D-: track 4.14 -> 21.3 mm, vias 0 -> 2
- net GND: track 104.6 -> 118.6 mm, vias 68 -> 71
- net +3V3: track 49.2 -> 62.8 mm, vias 36 -> 39
- net /Processor/ANALOG_IN_VYAW: track 0.00 -> 9.85 mm
- net /Processor/ANALOG_IN_VROLL: track 0.00 -> 9.78 mm
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Other:
- board text added: "ENCODERS"
- board text added: "RADIO"
- board text removed: "+3V3"
- board text removed: "+5V0"
- board text removed: "NRF24L01 RADIO"
- board text removed: "ROTARY ENCODERS"

Commit message: Finish first draft of v2.0 pcb
Parts:
- removed BZ1: Buzzer, Buzzer_Beeper:Buzzer_12x9.5RM7.6
- removed Q1: MMBT3904, Package_TO_SOT_SMD:SOT-23
- removed R43: 100, Resistor_SMD:R_0402_1005Metric
- removed R44: 1k, Resistor_SMD:R_0402_1005Metric
- moved J4 24.0 mm to (128.0, 112.6)
- moved C26 14.1 mm to (120.2, 94.7), turned to 180 degrees
- moved R99 6.34 mm to (130.9, 101.3), turned to 135 degrees
- moved R96 5.29 mm to (128.9, 116.9), turned to 270 degrees
- moved R67 4.40 mm to (131.6, 100.5), turned to 135 degrees
- moved R64 4.33 mm to (130.7, 97.4), turned to 180 degrees
- moved R89 2.87 mm to (140.9, 117.6)
- moved R91 2.87 mm to (140.9, 118.6)
- moved R59 1.95 mm to (140.9, 115.9)
- moved R65 1.95 mm to (140.9, 115.0)
- moved R88 0.52 mm to (142.4, 113.7)
- moved U4 0.19 mm to (125.9, 96.7)
- turned C57 to 315 degrees
Connections:
- U13 pad 58: /Human Machine Interface/PWM_Buzzer -> Net-(U13-Pad58)
Routing:
- net /Human Machine Interface/KEY_SCK: track 1.75 -> 90.3 mm, vias 1 -> 5
- net /Human Machine Interface/KEY_nSAMPLE: track 1.73 -> 67.6 mm, vias 1 -> 4
- net /Processor/USB_SENSE: track 17.1 -> 48.3 mm
- net /Human Machine Interface/ENC1_A: track 0.89 -> 31.6 mm, vias 1 -> 2
- net /Power Supply/USB_ID: track 22.9 -> 52.1 mm
- net /Power Supply/USB_D+: track 22.4 -> 51.4 mm
- net /Processor/KEY_MOSI: track 0.00 -> 28.5 mm
- net /Human Machine Interface/nRESET: track 8.07 -> 36.2 mm
- net /Power Supply/USB_D-: track 21.3 -> 48.8 mm
- net /Human Machine Interface/KEY_MISO: track 0.00 -> 26.5 mm, vias 0 -> 2
- net Net-(R91-Pad2): track 0.00 -> 26.4 mm, vias 0 -> 2
- net /Human Machine Interface/ENC1_B: track 0.89 -> 26.8 mm, vias 1 -> 2
- net Net-(R89-Pad1): track 0.00 -> 24.3 mm, vias 0 -> 2
- net /Human Machine Interface/ENC0_B: track 0.89 -> 24.3 mm, vias 1 -> 2
- net /Human Machine Interface/ENC0_A: track 0.89 -> 23.7 mm, vias 1 -> 2
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Other:
- board text added: "0"
- board text added: "3"
- board text added: "PTR"
- board text added: "Quadrotor Controller v2.0"
- board text added: "RESET"
- board text added: "RTR"
- board text added: "SER0"
- board text added: "SER1"
- board text added: "TTR"
- board text added: "YTR"
- board text removed: "+"
- board text removed: "-"
- board text removed: "ALARM"
- board text removed: "JTAG"
- board text removed: "PITCH TRIM"
- board text removed: "Piezo Buzzer"
- board text removed: "Quadrotor Controller v1.0 Specifications: STM32F446RE 1MB NOR Flash 32KB EEPROM NRF24L01 Flight Radio RN4871 Bluetooth Battery Charge/Protect USB JTAG"
- board text removed: "ROLL TRIM"
- board text removed: "STS LEDS"
- board text removed: "THROTTLE TRIM"
- board text removed: "YAW TRIM"
