File: hw/PCBDesign/HMIHardware.sch (KiCad schematic (older format))
At the start: 15 parts, among them U1 74HC165, U2 74HC165, U3 74HC165

Commit message: Work further on v2.0 of controller pcb
Changed lines of the file:
@@
 Text Label 9300 3400 0    50   ~ 0
 d3
+Text Label 9300 3600 0    50   ~ 0
+d15
+Text Label 9300 4150 0    50   ~ 0
+d14
+Text Label 9300 3700 0    50   ~ 0
+d13
+Text Label 9300 3800 0    50   ~ 0
+d12
 Text Label 9300 3500 0    50   ~ 0
-d15
+d8
 Text Label 9300 3200 0    50   ~ 0
-d14
+d9
 Text Label 9300 4250 0    50   ~ 0
-d13
+d10
 Text Label 9300 3300 0    50   ~ 0
-d12
-Text Label 9300 3600 0    50   ~ 0
-d8
-Text Label 9300 4150 0    50   ~ 0
-d9
-Text Label 9300 3700 0    50   ~ 0
-d10
-Text Label 9300 3800 0    50   ~ 0
 d11
 Text Label 9300 4050 0    50   ~ 0

Commit message: Finish first draft of v2.0 pcb
Connections:
- net labels removed: PWM_Buzzer
- wire segments 77 -> 75
Changed lines of the file:
@@
 $Descr A4 11693 8268
 encoding utf-8
-Sheet 2 11
+Sheet 2 10
 Title ""
 Date ""
@@
 $EndSheet
 $Sheet
-S 9600 5700 900  450
-U 60452CE3
-F0 "Audio Output" 50
-F1 "AudioOut.sch" 50
-F2 "V+" I L 9600 5850 50
-F3 "PWM_In" I L 9600 6000 50
-$EndSheet
-$Sheet
 S 9600 1650 900  1050
 U 60456C21
@@
 F5 "KeyUser" O L 9600 1900 50
 $EndSheet
-Text HLabel 9550 6000 0    50   Input ~ 0
-PWM_Buzzer
 Text HLabel 10650 850  2    50   Output ~ 0
 ENC0_A
@@
 Wire Wire Line
 	9500 4800 9600 4800
-Text HLabel 9550 5850 0    50   Input ~ 0
-V+
-Wire Wire Line
-	9550 6000 9600 6000
-Wire Wire Line
-	9550 5850 9600 5850
 Text HLabel 9450 3050 0    50   Input ~ 0
 V+
