File: hw/PCBDesign/ToggleSW.sch (KiCad schematic (older format))
At the start: 52 parts, among them J10 SW_B, J11 YTrim, J12 SW_C, J13 TTrim, J14 SW_D, J7 PTrim, J8 SW_A, J9 RTrim, SW10 UserSwitchD, SW3 PitchTrim, SW4 UserSwitchA, SW5 RollTrim, SW6 UserSwitchB, SW7 YawTrim, SW8 UserSwitchC, SW9 ThrottleTrim

Commit message: Start working on PCB rev 2.0
Parts:
- J10, J11, J12, J13, J14, J8, J9: footprint Connector_JST:JST_PH_B3B-PH-SM4-TB_1x03-1MP_P2.00mm_Vertical -> Connector_Molex:Molex_PicoBlade_53261-0371_1x03-1MP_P1.25mm_Horizontal; DigiKey 455-1735-2-ND -> WM7621CT-ND
- J7: footprint Connector_JST:JST_PH_B3B-PH-SM4-TB_1x03-1MP_P2.00mm_Vertical -> Connector_Molex:Molex_PicoBlade_53261-0371_1x03-1MP_P1.25mm_Horizontal; DigiKey 455-1735-2-ND -> WM7621CT-ND; Digikey (none) -> WM7621CT-ND
Changed lines of the file:
@@
 F 0 "J14" H 10030 3592 50  0000 L CNN
 F 1 "SW_D" H 10030 3501 50  0000 L CNN
-F 2 "Connector_JST:JST_PH_B3B-PH-SM4-TB_1x03-1MP_P2.00mm_Vertical" H 9950 3550 50  0001 C CNN
+F 2 "Connector_Molex:Molex_PicoBlade_53261-0371_1x03-1MP_P1.25mm_Horizontal" H 9950 3550 50  0001 C CNN
 F 3 "~" H 9950 3550 50  0001 C CNN
-F 4 "455-1735-2-ND" H 9950 3550 50  0001 C CNN "DigiKey"
+F 4 "WM7621CT-ND" H 9950 3550 50  0001 C CNN "DigiKey"
 	1    9950 3550
 	1    0    0    -1
@@
 F 0 "J12" H 7530 3592 50  0000 L CNN
 F 1 "SW_C" H 7530 3501 50  0000 L CNN
-F 2 "Connector_JST:JST_PH_B3B-PH-SM4-TB_1x03-1MP_P2.00mm_Vertical" H 7450 3550 50  0001 C CNN
+F 2 "Connector_Molex:Molex_PicoBlade_53261-0371_1x03-1MP_P1.25mm_Horizontal" H 7450 3550 50  0001 C CNN
 F 3 "~" H 7450 3550 50  0001 C CNN
-F 4 "455-1735-2-ND" H 7450 3550 50  0001 C CNN "DigiKey"
+F 4 "WM7621CT-ND" H 7450 3550 50  0001 C CNN "DigiKey"
 	1    7450 3550
 	1    0    0    -1
@@
 F 0 "J10" H 5080 3592 50  0000 L CNN
 F 1 "SW_B" H 5080 3501 50  0000 L CNN
-F 2 "Connector_JST:JST_PH_B3B-PH-SM4-TB_1x03-1MP_P2.00mm_Vertical" H 5000 3550 50  0001 C CNN
+F 2 "Connector_Molex:Molex_PicoBlade_53261-0371_1x03-1MP_P1.25mm_Horizontal" H 5000 3550 50  0001 C CNN
 F 3 "~" H 5000 3550 50  0001 C CNN
-F 4 "455-1735-2-ND" H 5000 3550 50  0001 C CNN "DigiKey"
+F 4 "WM7621CT-ND" H 5000 3550 50  0001 C CNN "DigiKey"
 	1    5000 3550
 	1    0    0    -1
@@
 F 0 "J8" H 2680 3592 50  0000 L CNN
 F 1 "SW_A" H 2680 3501 50  0000 L CNN
-F 2 "Connector_JST:JST_PH_B3B-PH-SM4-TB_1x03-1MP_P2.00mm_Vertical" H 2600 3550 50  0001 C CNN
+F 2 "Connector_Molex:Molex_PicoBlade_53261-0371_1x03-1MP_P1.25mm_Horizontal" H 2600 3550 50  0001 C CNN
 F 3 "~" H 2600 3550 50  0001 C CNN
-F 4 "455-1735-2-ND" H 2600 3550 50  0001 C CNN "DigiKey"
+F 4 "WM7621CT-ND" H 2600 3550 50  0001 C CNN "DigiKey"
 	1    2600 3550
 	1    0    0    -1
@@
 F 0 "J7" V 1864 930 50  0000 L CNN
 F 1 "PTrim" V 1773 930 50  0000 L CNN
-F 2 "Connector_JST:JST_PH_B3B-PH-SM4-TB_1x03-1MP_P2.00mm_Vertical" H 1900 750 50  0001 C CNN
+F 2 "Connector_Molex:Molex_PicoBlade_53261-0371_1x03-1MP_P1.25mm_Horizontal" H 1900 750 50  0001 C CNN
 F 3 "~" H 1900 750 50  0001 C CNN
-F 4 "455-1735-2-ND" H 1900 750 50  0001 C CNN "DigiKey"
+F 4 "WM7621CT-ND" H 1900 750 50  0001 C CNN "DigiKey"
+F 5 "WM7621CT-ND" H 1900 750 50  0001 C CNN "Digikey"
 	1    1900 750
 	0    1    -1   0
@@
 F 0 "J9" V 4364 930 50  0000 L CNN
 F 1 "RTrim" V 4273 930 50  0000 L CNN
-F 2 "Connector_JST:JST_PH_B3B-PH-SM4-TB_1x03-1MP_P2.00mm_Vertical" H 4400 750 50  0001 C CNN
+F 2 "Connector_Molex:Molex_PicoBlade_53261-0371_1x03-1MP_P1.25mm_Horizontal" H 4400 750 50  0001 C CNN
 F 3 "~" H 4400 750 50  0001 C CNN
-F 4 "455-1735-2-ND" H 4400 750 50  0001 C CNN "DigiKey"
+F 4 "WM7621CT-ND" H 4400 750 50  0001 C CNN "DigiKey"
 	1    4400 750
 	0    1    -1   0
@@
 F 0 "J11" V 6814 930 50  0000 L CNN
 F 1 "YTrim" V 6723 930 50  0000 L CNN
-F 2 "Connector_JST:JST_PH_B3B-PH-SM4-TB_1x03-1MP_P2.00mm_Vertical" H 6850 750 50  0001 C CNN
+F 2 "Connector_Molex:Molex_PicoBlade_53261-0371_1x03-1MP_P1.25mm_Horizontal" H 6850 750 50  0001 C CNN
 F 3 "~" H 6850 750 50  0001 C CNN
-F 4 "455-1735-2-ND" H 6850 750 50  0001 C CNN "DigiKey"
+F 4 "WM7621CT-ND" H 6850 750 50  0001 C CNN "DigiKey"
 	1    6850 750
 	0    1    -1   0
@@
 F 0 "J13" V 9264 930 50  0000 L CNN
 F 1 "TTrim" V 9173 930 50  0000 L CNN
-F 2 "Connector_JST:JST_PH_B3B-PH-SM4-TB_1x03-1MP_P2.00mm_Vertical" H 9300 750 50  0001 C CNN
+F 2 "Connector_Molex:Molex_PicoBlade_53261-0371_1x03-1MP_P1.25mm_Horizontal" H 9300 750 50  0001 C CNN
 F 3 "~" H 9300 750 50  0001 C CNN
-F 4 "455-1735-2-ND" H 9300 750 50  0001 C CNN "DigiKey"
+F 4 "WM7621CT-ND" H 9300 750 50  0001 C CNN "DigiKey"
 	1    9300 750
 	0    1    -1   0
